File: LightingNodeProV2/LightingNodeProV2.kicad_pcb (KiCad board)
At the start: 2 copper layers, 45 x 35 mm, 6 parts, among them J1 sata15, J2 Conn_01x03, J3 Conn_01x03, U1 ProMicro_ProMicro

Commit message: edit
Other:
- rule pad_to_mask_clearance: 0.051 -> 0
Changed lines of the file:
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@@
       (dielectric_constraints no)
     )
-    (pad_to_mask_clearance 0.051)
-    (solder_mask_min_width 0.25)
+    (pad_to_mask_clearance 0)
     (aux_axis_origin 144 97)
     (grid_origin 144 97)
@@
     (pts (xy 166.92 75.68) (xy 121.92 75.68))
     (height 9)
-    (gr_text "45,0000 mm" (at 144.42 65.53) (layer "Dwgs.User")
+    (gr_text "45.0000 mm" (at 144.42 65.53) (layer "Dwgs.User")
       (effects (font (size 1 1) (thickness 0.15)))
     )
@@
     (pts (xy 121.92 106.68) (xy 125.92 106.68))
     (height 10)
-    (gr_text "4,0000 mm" (at 123.92 115.53) (layer "Dwgs.User")
+    (gr_text "4.0000 mm" (at 123.92 115.53) (layer "Dwgs.User")
       (effects (font (size 1 1) (thickness 0.15)))
     )
@@
     (pts (xy 166.92 79.68) (xy 162.92 79.68))
     (height 8)
-    (gr_text "4,0000 mm" (at 164.92 70.53) (layer "Dwgs.User")
+    (gr_text "4.0000 mm" (at 164.92 70.53) (layer "Dwgs.User")
       (effects (font (size 1 1) (thickness 0.15)))
     )
@@
     (pts (xy 166.92 110.68) (xy 166.92 75.68))
     (height 11)
-    (gr_text "35,0000 mm" (at 176.77 93.18 90) (layer "Dwgs.User")
+    (gr_text "35.0000 mm" (at 176.77 93.18 90) (layer "Dwgs.User")
       (effects (font (size 1 1) (thickness 0.15)))
     )
@@
     (pts (xy 125.92 110.68) (xy 125.92 106.68))
     (height -13)
-    (gr_text "4,0000 mm" (at 111.77 108.68 90) (layer "Dwgs.User")
+    (gr_text "4.0000 mm" (at 111.77 108.68 90) (layer "Dwgs.User")
       (effects (font (size 1 1) (thickness 0.15)))
     )
@@
     (pts (xy 162.92 75.68) (xy 162.92 79.68))
     (height -10)
-    (gr_text "4,0000 mm" (at 171.77 77.68 90) (layer "Dwgs.User")
+    (gr_text "4.0000 mm" (at 171.77 77.68 90) (layer "Dwgs.User")
       (effects (font (size 1 1) (thickness 0.15)))
     )
@@
   (segment (start 143.24 102.34) (end 143.24 106.6) (width 1) (layer "B.Cu") (net 2))
   (segment (start 165.1 108.14) (end 165.1 87.82) (width 1) (layer "B.Cu") (net 2))
-  (segment (start 137.16 97.98) (end 157.48 97.98) (width 0.75) (layer "F.Cu") (net 3))
-  (segment (start 157.98 103.06) (end 160.02 103.06) (width 0.75) (layer "F.Cu") (net 3))
-  (segment (start 135.89 96.71) (end 137.16 97.98) (width 0.75) (layer "F.Cu") (net 3))
-  (segment (start 135.89 94.17) (end 135.89 96.71) (width 0.75) (layer "F.Cu") (net 3))
-  (segment (start 157.98 98.48) (end 157.98 103.06) (width 0.75) (layer "F.Cu") (net 3))
-  (segment (start 157.48 97.98) (end 157.98 98.48) (width 0.75) (layer "F.Cu") (net 3))
-  (segment (start 139.7 90.36) (end 160.02 90.36) (width 0.75) (layer "F.Cu") (net 4))
-  (segment (start 138.43 91.63) (end 139.7 90.36) (width 0.75) (layer "F.Cu") (net 4))
-  (segment (start 138.43 94.17) (end 138.43 91.63) (width 0.75) (layer "F.Cu") (net 4))
+  (segment (start 137.16 97.98) (end 157.48 97.98) (width 0.75) (layer "B.Cu") (net 3))
+  (segment (start 157.98 103.06) (end 160.02 103.06) (width 0.75) (layer "B.Cu") (net 3))
+  (segment (start 135.89 96.71) (end 137.16 97.98) (width 0.75) (layer "B.Cu") (net 3))
+  (segment (start 135.89 94.17) (end 135.89 96.71) (width 0.75) (layer "B.Cu") (net 3))
+  (segment (start 157.98 98.48) (end 157.98 103.06) (width 0.75) (layer "B.Cu") (net 3))
+  (segment (start 157.48 97.98) (end 157.98 98.48) (width 0.75) (layer "B.Cu") (net 3))
+  (segment (start 139.7 90.36) (end 160.02 90.36) (width 0.75) (layer "B.Cu") (net 4))
+  (segment (start 138.43 91.63) (end 139.7 90.36) (width 0.75) (layer "B.Cu") (net 4))
+  (segment (start 138.43 94.17) (end 138.43 91.63) (width 0.75) (layer "B.Cu") (net 4))
   (zone (net 1) (net_name "/GND") (layer "F.Cu") (name "gnd") (hatch edge 0.5)
     (connect_pads (clearance 0.508))
